Commit message: FUNCTIONING: single door with revolute joint

File: simulation/flexible_environment/urdf/flexible_window.xacro (robot description, xacro)
@@ -1,25 +1,32 @@
 <?xml version="1.0"?>
 <robot name="window_environment" xmlns:xacro="http://www.ros.org/wiki/xacro">
+	<xacro:arg name="mass" default="1"/>
   <!-- Used for fixing robot to Gazebo 'base_link' -->
   <link name="world"/>
-	<joint name="window_hinge_1" type="revolute">
+	<joint name="window_hinge_1" type="continuous">
     <parent link="world"/>
     <child link="window_1"/>
-    <origin xyz="0 0.225 1.125"/>
-    <axis xyz="0 0 1"/>
-    <limit effort="15.0" lower="-1.57" upper="1.57" velocity="1"/>
+    <origin xyz="0 0 1"/>
+    <axis xyz="1 0 0"/>
+		<!-- <limit effort="10.0" velocity="10.0" /> -->
   </joint>
   <link name="window_1">
      <inertial>
-      <origin xyz="0 0.2 1.125"/>
-      <mass value="5.0" />
-      <inertia  ixx="1.0" ixy="0.0"  ixz="0.0"  iyy="100.0"  iyz="0.0"  izz="1.0" />
+      <origin xyz="0 0.5 1"/>
+      <mass value="$(arg mass)" />
+      <inertia  ixx="${$(arg mass)*1/12/1.01}" ixy="0.0"  ixz="0.0"  iyy="${$(arg mass)*1/12/1.01}"  iyz="0.0"  izz="${$(arg mass)*1/6}" />
     </inertial>
     <visual>
-      <origin xyz="0 0.2 1.125" rpy="0 0 1.57" />
+      <origin xyz="0 0.5 0.05" rpy="0 0 0" />
       <geometry>
-        <box size="0.4 .1 2.2"/>
+        <box size="1.0 1.0 0.1"/>
       </geometry>
     </visual>
+		<collision>
+      <origin xyz="0 0.5 0.05" rpy="0 0 0" />
+      <geometry>
+        <box size="1.0 1.0 0.1"/>
+      </geometry>
+		</collision>
   </link>
 </robot>

Commit message: 5 rigid windows in line: new version of urdf with updated .xacro and .gazebo file

File: simulation/flexible_environment/urdf/flexible_window.xacro (robot description, xacro)
@@ -1,32 +1,49 @@
-<?xml version="1.0"?>
-<robot name="window_environment" xmlns:xacro="http://www.ros.org/wiki/xacro">
-	<xacro:arg name="mass" default="1"/>
-  <!-- Used for fixing robot to Gazebo 'base_link' -->
-  <link name="world"/>
-	<joint name="window_hinge_1" type="continuous">
-    <parent link="world"/>
-    <child link="window_1"/>
-    <origin xyz="0 0 1"/>
-    <axis xyz="1 0 0"/>
-		<!-- <limit effort="10.0" velocity="10.0" /> -->
-  </joint>
-  <link name="window_1">
-     <inertial>
-      <origin xyz="0 0.5 1"/>
-      <mass value="$(arg mass)" />
-      <inertia  ixx="${$(arg mass)*1/12/1.01}" ixy="0.0"  ixz="0.0"  iyy="${$(arg mass)*1/12/1.01}"  iyz="0.0"  izz="${$(arg mass)*1/6}" />
-    </inertial>
-    <visual>
-      <origin xyz="0 0.5 0.05" rpy="0 0 0" />
-      <geometry>
-        <box size="1.0 1.0 0.1"/>
-      </geometry>
-    </visual>
-		<collision>
-      <origin xyz="0 0.5 0.05" rpy="0 0 0" />
-      <geometry>
-        <box size="1.0 1.0 0.1"/>
-      </geometry>
-		</collision>
-  </link>
+<?xml version="1.0" ?>
+<robot xmlns:xacro="http://www.ros.org/wiki/xacro">
+	<xacro:arg name="mass" default="0.1"/>
+  <xacro:arg name="stiffness" default="0.2"/>
+  <xacro:arg name="damping" default="0.03"/>
+  <xacro:property name="offset" value="3"/>
+	<xacro:property name="length" value="2"/>
+	<xacro:property name="width" value="2"/>
+  <xacro:property name="height" value="0.1"/>
+  <xacro:property name="space_between" value="${0.2+width}"/>
+	<xacro:property name="upper_limit" value="90"/>
+	<xacro:property name="lower_limit" value="-270"/>
+  <xacro:property name="mass" value="$(arg mass)"/>
+  <xacro:property name="friction" default="${mass*0.01}"/>
+	<xacro:property name="stiffness" default="$(arg stiffness)"/>
+  <xacro:property name="damping" default="$(arg damping)"/>
+  <xacro:macro name="window" params="number">
+    <link name="window_${number}">
+      <inertial>
+        <origin xyz="0 ${width/2} 0"/>
+        <mass value="${mass}" />
+        <inertia  ixx="${1/12*mass*(height**2+width**2)+1/4*mass*length**2}" ixy="0.0"  ixz="0.0"
+                  iyy="${1/12*mass*(height**2+length**2)}"  iyz="0.0"  izz="${1/12*mass*(width**2+length**2)}" />
+      </inertial>
+      <visual>
+        <origin xyz="0 ${width/2} 0"/>
+        <geometry>
+          <box size="${length} ${width} ${height}"/>
+        </geometry>
+      </visual>
+      <collision>
+        <origin xyz="0 ${width/2} 0"/>
+        <geometry>
+          <box size="${length} ${width} ${height}"/>
+        </geometry>
+      </collision>
+    </link>
+    <joint name="hinge_${number}" type="revolute">
+      <parent link="world"/>
+      <child link="window_${number}"/>
+      <dynamics damping="${damping}" friction="${friction}" />
+      <origin xyz="0 0 ${offset+(number-1)*space_between}"/>
+      <axis xyz="1 0 0"/>
+      <limit lower="${lower_limit*pi/180}" upper="${upper_limit*pi/180}" effort="1000.0" velocity="100.0"/>
+    </joint>
+    <!-- Import all Gazebo-customization elements, including Gazebo colors -->
+    <xacro:include filename="$(find flexible_environment)/urdf/flexible_window.gazebo"/>
+  </xacro:macro>
 </robot>
